Commit message: 2803 lecture from home

File: src/simple4wheeler/model/simple4wheeler.xacro (robot description, xacro)
@@ -1,4 +1,4 @@
 <robot name="simple4wheeler" xmlns:xacro="http://www.ros.org/wiki/xacro">
-    <xacro:property name="pi" value="3.142" />
+    <xacro:property name="pi_" value="3.142" />
     <link name="map">
     </link>
@@ -31,3 +31,93 @@
         <child link="link_chassis"/>
     </joint>
+    <link name="link_right_back_wheel">
+        <inertial>
+            <mass value="0.2"/>
+            <origin rpy="0 0 0" xyz="0 0 0.1"/>
+                <inertia ixx="0.00052"
+                         ixy="0"
+                         ixz="0"
+                         iyy="0.00052"
+                         iyz="0"
+                         izz="0.001" />
+        </inertial>
+        <collision name="collision_right_back_wheel">
+            <geometry>
+                <cylinder length="0.04" radius="0.3"/>
+            </geometry>
+        </collision>
+        <visual name="visual_right_back_wheel">
+            <geometry>
+                <cylinder length="0.04" radius="0.3"/>
+            </geometry>
+        </visual>
+    </link>
+    <joint name="joint_right_back_wheel" type="continuous">
+        <origin rpy="0 0 0" xyz="0 0 0" />
+        <parent link="link_chassis" />
+        <child link="link_right_back_wheel" />
+        <axis rpy="0 0 0" xyz="0 0 1" />
+        <limit effort="10" velocity="10" />
+        <joint_properties damping="1.0" friction="1.0" />
+    </joint>
+    <link name="link_lidar">
+        <inertial>
+            <mass value="0.1"/>
+            <origin rpy="0 0 0" xyz="0 0 0"/>
+                <inertia ixx="0.00001"
+                         ixy="0"
+                         ixz="0"
+                         iyy="0.00001"
+                         iyz="0"
+                         izz="0.00001" />
+        </inertial>
+        <collision name="collision_lidar">
+            <geometry>
+                <box size="0.07 0.07 0.07" />
+            </geometry>
+        </collision>
+        <visual name="visual_lidar">
+            <geometry>
+                <mesh filename="file://package://simple4wheeler/model/rplidar_a2_simple.stl" />
+            </geometry>
+        </visual>
+    </link>
+    <joint name="joint_lidar" type="fixed">
+        <origin rpy="0 0 0" xyz="0 0 0.07" />
+        <parent link="link_chassis" />
+        <child link="link_lidar" />
+    </joint>
+    <gazebo reference="link_lidar">
+        <sensor type="ray" name="sensor_lidar">
+            <update_rate>10</update_rate>
+            <visualize>true</visualize>
+            <ray>
+                <scan>
+                    <horizontal>
+                        <samples>400</samples>
+                        <min_angle>-${pi_}</min_angle>
+                        <max_angle>${pi_}</max_angle>
+                    </horizontal>
+                    <vertical>
+                        <samples>1</samples>
+                        <min_angle>-0.05</min_angle>
+                        <max_angle>0.05</max_angle>
+                    </vertical>
+                </scan>
+                    <range>
+                        <min>0.015</min>
+                        <max>12</max>
+                        <resolution>0.01</resolution>
+                    </range>
+            </ray>
+            <plugin name="gazebo_ros_lidar" filename="libgazebo_ros_laser.so">
+                <gaussianNoise>0.01</gaussianNoise>
+                <updateRate>10</updateRate>
+                <topicName>lidar</topicName>
+                <minRange>0.15</minRange>
+                <maxRange>12.0</maxRange>
+                <frameName>link_lidar</frameName>
+            </plugin>
+        </sensor>
+</gazebo>
 </robot>
